File: range_tag.sch (EAGLE design)
At the start: 26 parts, among them U1 FT232RL-BASICSSOP, U2 MCP73833, U3 ESP8266-12E/ESP-12E

Commit message: M
Connections:
- net N$1 renamed USBDM
- net N$2 renamed USBDP
Changed lines of the file:
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@@
 </segment>
 </net>
-<net name="N$1" class="0">
+<net name="USBDM" class="0">
 <segment>
 <pinref part="JP2" gate="G$1" pin="D-"/>
@@
 </segment>
 </net>
-<net name="N$2" class="0">
+<net name="USBDP" class="0">
 <segment>
 <pinref part="U1" gate="G$1" pin="USBDP"/>

Commit message: Ok
Parts:
- removed C2: (no value), SparkFun-Capacitors:CAP0805
- renumbered J1 to BATT, U2 to MCP73833
Connections:
- net N$13 renamed N_PG
- net N$5 renamed STAT1
- net N$6 renamed STAT2
- removed net 3V3: C2.1, U$2.OUT, U1.3V3OUT
- new net 3V3_USB: U1.3V3OUT
- net +3V3: now also U$2.OUT
- net GND: no longer C2.2
Changed lines of the file:
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@@
 <part name="SUPPLY3" library="supply2" library_urn="urn:adsk.eagle:library:372" deviceset="GND" device=""/>
 <part name="C1" library="SparkFun-Capacitors" deviceset="CAP" device="0805"/>
-<part name="C2" library="SparkFun-Capacitors" deviceset="CAP" device="0805"/>
 <part name="SUPPLY4" library="supply2" library_urn="urn:adsk.eagle:library:372" deviceset="GND" device=""/>
-<part name="SUPPLY5" library="supply2" library_urn="urn:adsk.eagle:library:372" deviceset="GND" device=""/>
 <part name="C3" library="SparkFun-Capacitors" deviceset="CAP_POL" device="1206-KIT"/>
 <part name="SUPPLY6" library="supply2" library_urn="urn:adsk.eagle:library:372" deviceset="GND" device=""/>
@@
 <part name="SUPPLY9" library="SparkFun-Aesthetics" deviceset="5V" device=""/>
 <part name="SUPPLY10" library="SparkFun-Aesthetics" deviceset="5V" device=""/>
-<part name="U2" library="SparkFun-PowerIC" deviceset="MCP73833" device=""/>
+<part name="MCP73833" library="SparkFun-PowerIC" deviceset="MCP73833" device=""/>
 <part name="SUPPLY11" library="SparkFun-Aesthetics" deviceset="5V" device=""/>
 <part name="SUPPLY12" library="supply2" library_urn="urn:adsk.eagle:library:372" deviceset="GND" device=""/>
@@
 <part name="R5" library="SparkFun-Resistors" deviceset="RESISTOR" device="1206" value="1K"/>
 <part name="SUPPLY15" library="SparkFun-Aesthetics" deviceset="5V" device=""/>
-<part name="J1" library="SparkFun-Connectors" deviceset="JST_2MM_MALE" device=""/>
+<part name="BATT" library="SparkFun-Connectors" deviceset="JST_2MM_MALE" device=""/>
 <part name="SUPPLY16" library="supply2" library_urn="urn:adsk.eagle:library:372" deviceset="GND" device=""/>
 <part name="R6" library="SparkFun-Resistors" deviceset="RESISTOR" device="1206" value="2K"/>
@@
 <instance part="SUPPLY3" gate="GND" x="-53.34" y="116.84"/>
 <instance part="C1" gate="G$1" x="-43.18" y="124.46"/>
-<instance part="C2" gate="G$1" x="-22.86" y="124.46"/>
 <instance part="SUPPLY4" gate="GND" x="-43.18" y="116.84"/>
-<instance part="SUPPLY5" gate="GND" x="-22.86" y="116.84"/>
 <instance part="C3" gate="G$1" x="-33.02" y="127"/>
 <instance part="SUPPLY6" gate="GND" x="-33.02" y="116.84"/>
@@
 <instance part="SUPPLY9" gate="G$1" x="30.48" y="149.86"/>
 <instance part="SUPPLY10" gate="G$1" x="40.64" y="149.86"/>
-<instance part="U2" gate="G$1" x="124.46" y="137.16"/>
+<instance part="MCP73833" gate="G$1" x="124.46" y="137.16"/>
 <instance part="SUPPLY11" gate="G$1" x="99.06" y="170.18"/>
 <instance part="SUPPLY12" gate="GND" x="99.06" y="111.76"/>
@@
 <instance part="R5" gate="G$1" x="63.5" y="147.32" rot="R90"/>
 <instance part="SUPPLY15" gate="G$1" x="63.5" y="170.18"/>
-<instance part="J1" gate="G$1" x="203.2" y="144.78" rot="MR90"/>
+<instance part="BATT" gate="G$1" x="203.2" y="144.78" rot="MR90"/>
 <instance part="SUPPLY16" gate="GND" x="190.5" y="111.76"/>
 <instance part="R6" gate="G$1" x="160.02" y="124.46" rot="R90"/>
@@
 <pinref part="U3" gate="G$1" pin="VCC"/>
 </segment>
+<segment>
+<pinref part="U$2" gate="G$1" pin="OUT"/>
+<wire x1="218.44" y1="127" x2="220.98" y2="127" width="0.1524" layer="91"/>
+<label x="220.98" y="127" size="1.778" layer="95"/>
+</segment>
 </net>
 <net name="GND" class="0">
@@
 <pinref part="SUPPLY4" gate="GND" pin="GND"/>
 <wire x1="-43.18" y1="121.92" x2="-43.18" y2="119.38" width="0.1524" layer="91"/>
-</segment>
-<segment>
-<pinref part="C2" gate="G$1" pin="2"/>
-<pinref part="SUPPLY5" gate="GND" pin="GND"/>
-<wire x1="-22.86" y1="121.92" x2="-22.86" y2="119.38" width="0.1524" layer="91"/>
 </segment>
 <segment>
@@
 </segment>
 <segment>
-<pinref part="U2" gate="G$1" pin="VSS"/>
+<pinref part="MCP73833" gate="G$1" pin="VSS"/>
 <wire x1="109.22" y1="124.46" x2="99.06" y2="124.46" width="0.1524" layer="91"/>
 <wire x1="99.06" y1="124.46" x2="99.06" y2="114.3" width="0.1524" layer="91"/>
@@
 </segment>
 <segment>
-<pinref part="J1" gate="G$1" pin="-"/>
+<pinref part="BATT" gate="G$1" pin="-"/>
 <pinref part="SUPPLY16" gate="GND" pin="GND"/>
 <wire x1="198.12" y1="144.78" x2="190.5" y2="144.78" width="0.1524" layer="91"/>
@@
 <pinref part="C5" gate="G$1" pin="2"/>
 <wire x1="58.42" y1="35.56" x2="58.42" y2="38.1" width="0.1524" layer="91"/>
-</segment>
-</net>
-<net name="3V3" class="0">
-<segment>
-<wire x1="-12.7" y1="132.08" x2="-22.86" y2="132.08" width="0.1524" layer="91"/>
-<pinref part="C2" gate="G$1" pin="1"/>
-<wire x1="-22.86" y1="132.08" x2="-22.86" y2="129.54" width="0.1524" layer="91"/>
-<label x="-20.32" y="132.08" size="1.778" layer="95"/>
-<pinref part="U1" gate="G$1" pin="3V3OUT"/>
-</segment>
-<segment>
-<pinref part="U$2" gate="G$1" pin="OUT"/>
-<wire x1="218.44" y1="127" x2="220.98" y2="127" width="0.1524" layer="91"/>
-<label x="220.98" y="127" size="1.778" layer="95"/>
 </segment>
 </net>
@@
 </segment>
 <segment>
-<pinref part="U2" gate="G$1" pin="VDD@1"/>
+<pinref part="MCP73833" gate="G$1" pin="VDD@1"/>
 <pinref part="SUPPLY11" gate="G$1" pin="5V"/>
 <wire x1="109.22" y1="147.32" x2="99.06" y2="147.32" width="0.1524" layer="91"/>
 <wire x1="99.06" y1="147.32" x2="99.06" y2="170.18" width="0.1524" layer="91"/>
-<pinref part="U2" gate="G$1" pin="VDD@2"/>
+<pinref part="MCP73833" gate="G$1" pin="VDD@2"/>
 <wire x1="109.22" y1="144.78" x2="99.06" y2="144.78" width="0.1524" layer="91"/>
 <wire x1="99.06" y1="144.78" x2="99.06" y2="147.32" width="0.1524" layer="91"/>
@@
 </segment>
 </net>
-<net name="N$5" class="0">
-<segment>
-<pinref part="U2" gate="G$1" pin="STAT1"/>
+<net name="STAT1" class="0">
+<segment>
+<pinref part="MCP73833" gate="G$1" pin="STAT1"/>
 <wire x1="109.22" y1="137.16" x2="86.36" y2="137.16" width="0.1524" layer="91"/>
 <pinref part="R3" gate="G$1" pin="1"/>
@@
 </segment>
 </net>
-<net name="N$6" class="0">
-<segment>
-<pinref part="U2" gate="G$1" pin="STAT2"/>
+<net name="STAT2" class="0">
+<segment>
+<pinref part="MCP73833" gate="G$1" pin="STAT2"/>
 <wire x1="109.22" y1="134.62" x2="76.2" y2="134.62" width="0.1524" layer="91"/>
 <pinref part="R4" gate="G$1" pin="1"/>
@@
 </segment>
 </net>
-<net name="N$13" class="0">
+<net name="N_PG" class="0">
 <segment>
 <pinref part="R5" gate="G$1" pin="1"/>
 <wire x1="63.5" y1="132.08" x2="63.5" y2="142.24" width="0.1524" layer="91"/>
-<pinref part="U2" gate="G$1" pin="~PG"/>
+<pinref part="MCP73833" gate="G$1" pin="~PG"/>
 <wire x1="109.22" y1="132.08" x2="63.5" y2="132.08" width="0.1524" layer="91"/>
 </segment>
@@
 <net name="V_BATT" class="0">
 <segment>
-<pinref part="U2" gate="G$1" pin="VBAT@2"/>
+<pinref part="MCP73833" gate="G$1" pin="VBAT@2"/>
 <wire x1="139.7" y1="147.32" x2="144.78" y2="147.32" width="0.1524" layer="91"/>
-<pinref part="U2" gate="G$1" pin="VBAT@1"/>
+<pinref part="MCP73833" gate="G$1" pin="VBAT@1"/>
 <wire x1="139.7" y1="144.78" x2="144.78" y2="144.78" width="0.1524" layer="91"/>
 <wire x1="144.78" y1="144.78" x2="144.78" y2="147.32" width="0.1524" layer="91"/>
 <junction x="144.78" y="147.32"/>
-<pinref part="J1" gate="G$1" pin="+"/>
+<pinref part="BATT" gate="G$1" pin="+"/>
 <wire x1="144.78" y1="147.32" x2="193.04" y2="147.32" width="0.1524" layer="91"/>
 <pinref part="C4" gate="G$1" pin="1"/>
@@
 <net name="N$16" class="0">
 <segment>
-<pinref part="U2" gate="G$1" pin="PROG"/>
+<pinref part="MCP73833" gate="G$1" pin="PROG"/>
 <pinref part="R6" gate="G$1" pin="2"/>
 <wire x1="139.7" y1="129.54" x2="160.02" y2="129.54" width="0.1524" layer="91"/>
@@
 <net name="N$7" class="0">
 <segment>
-<pinref part="U2" gate="G$1" pin="THERM"/>
+<pinref part="MCP73833" gate="G$1" pin="THERM"/>
 <pinref part="RT1" gate="G$1" pin="2"/>
 <wire x1="139.7" y1="137.16" x2="160.02" y2="137.16" width="0.1524" layer="91"/>
@@
 </segment>
 </net>
+<net name="3V3_USB" class="0">
+<segment>
+<wire x1="-12.7" y1="132.08" x2="-22.86" y2="132.08" width="0.1524" layer="91"/>
+<label x="-22.86" y="132.08" size="1.778" layer="95"/>
+<pinref part="U1" gate="G$1" pin="3V3OUT"/>
+</segment>
+</net>
