File: range_tag.brd (EAGLE design)
At the start: 72 x 44 mm, 26 parts, among them U1 FT232RL-BASICSSOP, U2 MCP73833, U3 ESP8266-12E/ESP-12E

Commit message: more
Parts:
- moved U$2 13.1 mm to (17.9, 27.0), flipped to the bottom, turned to 0 degrees
- moved J1 11.0 mm to (8.45, 23.7)
- moved RT1 5.83 mm to (24.5, 36.9)
- moved D5 5.78 mm to (7.91, 31.9), turned to 180 degrees
- moved R5 5.78 mm to (7.91, 31.9), turned to 0 degrees
- moved D4 5.58 mm to (7.91, 37.6), turned to 180 degrees
- moved R3 5.58 mm to (7.91, 37.6), turned to 0 degrees
- moved C4 3.24 mm to (18.6, 36.9)
- moved U2 3.06 mm to (17.7, 32.3)
- moved RT2 3.03 mm to (28.5, 35.5), turned to 270 degrees
- moved R9 2.39 mm to (32.7, 35.5), turned to 270 degrees
- moved R6 0.73 mm to (24.5, 34.2)
- moved D3 0.21 mm to (7.91, 34.8), turned to 180 degrees
- moved R4 0.21 mm to (7.91, 34.8), turned to 0 degrees
Routing:
- net N$8: track 0.00 -> 9.46 mm, vias 0 -> 1
- net N$7: track 0.00 -> 7.25 mm
- net 5V: track 12.9 -> 16.5 mm, vias 1 -> 4
- net GND: track 0.00 -> 2.60 mm, vias 0 -> 1
- net N$16: track 5.96 -> 5.31 mm

Commit message: M
Parts:
- moved C2 8.04 mm to (7.64, 19.1)
- moved C1 7.35 mm to (9.58, 19.0), turned to 270 degrees
- moved C3 6.97 mm to (11.9, 17.3)
- moved C5 6.15 mm to (40.3, 25.9)
- moved U$2 5.44 mm to (21.7, 30.9)
- moved D1 3.09 mm to (20.2, 7.78)
- moved R1 3.06 mm to (20.2, 7.78)
- moved C4 2.50 mm to (21.0, 36.0), turned to 270 degrees
- moved R2 2.33 mm to (17.6, 7.86)
- moved D2 2.29 mm to (17.7, 7.89)
- moved U1 1.93 mm to (10.6, 25.2), turned to 180 degrees
- moved JP1 1.67 mm to (43.5, 27.5)
- moved U2 0.81 mm to (17.0, 32.7), flipped to the bottom, turned to 180 degrees
- moved JP2 0.52 mm to (10.6, 10.9), flipped to the bottom, turned to 90 degrees
Connections:
- net N$1 renamed USBDM
- net N$2 renamed USBDP
Routing:
- net N$8: track 9.46 -> 0.00 mm, vias 1 -> 0
- net N$7: track 7.25 -> 0.00 mm
- net 5V: track 16.5 -> 9.87 mm, vias 4 -> 3
- net N$16: track 5.31 -> 0.00 mm
- net GND: track 2.60 -> 0.00 mm, vias 1 -> 0
- net V_BATT: track 2.48 -> 0.00 mm
- added copper zone on layer 16, net 3V3
- added copper zone on layer 1, net GND

Commit message: Ok
Parts:
- removed C2: (no value), SparkFun-Capacitors:0805
- removed J1: (no value), SparkFun-Connectors:JST-2-SMD
- removed U2: MCP73833, SparkFun-PowerIC:MSOP-10
- added BATT: (no value), SparkFun-Connectors:JST-2-SMD
- added MCP73833: MCP73833, SparkFun-PowerIC:MSOP-10
- moved C3 8.96 mm to (10.00, 26.1), flipped to the bottom, turned to 180 degrees
- moved R6 8.65 mm to (16.0, 32.6), turned to 0 degrees
- moved RT1 7.24 mm to (21.0, 30.5), turned to 90 degrees
- moved U$2 5.22 mm to (25.0, 26.9), turned to 180 degrees
- moved C1 4.83 mm to (9.22, 23.8), flipped to the bottom, turned to 0 degrees
- moved C5 4.52 mm to (36.0, 24.4), flipped to the bottom
- moved JP1 2.71 mm to (43.2, 24.8)
- moved U1 1.69 mm to (11.3, 23.7)
- moved U3 1.27 mm to (31.4, 17.2)
- moved R9 0.46 mm to (33.1, 35.5), turned to 90 degrees
- moved C4 0.27 mm to (21.0, 35.7)
- moved D1 0.20 mm to (20.0, 7.88)
- moved RT2 0.19 mm to (28.3, 35.6), turned to 90 degrees
- moved JP2 0.18 mm to (10.6, 10.7)
- moved R1 0.17 mm to (20.0, 7.88)
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Connections:
- removed net 3V3: C2.1, U$2.1, U1.17
- removed net N$13: R5.1, U2.7
- removed net N$5: R3.1, U2.3
- removed net N$6: R4.1, U2.4
- new net 3V3_USB: U1.17
- new net N_PG: MCP73833.7, R5.1
- new net STAT1: MCP73833.3, R3.1
- new net STAT2: MCP73833.4, R4.1
- net +3V3: now also U$2.1
- net 5V: now also MCP73833.1, MCP73833.2; no longer U2.1, U2.2
- net GND: now also BATT.1, MCP73833.5; no longer C2.2, J1.1, U2.5
- net N$16: now also MCP73833.6; no longer U2.6
- net N$7: now also MCP73833.8; no longer U2.8
- net V_BATT: now also BATT.2, MCP73833.10, MCP73833.9; no longer J1.2, U2.10, U2.9
Routing:
- net MOSI: track 0.00 -> 51.9 mm, vias 0 -> 1
- net SPICLK: track 0.00 -> 51.1 mm, vias 0 -> 1
- net MISO: track 0.00 -> 48.5 mm, vias 0 -> 1
- net SPISS: track 0.00 -> 47.0 mm, vias 0 -> 1
- net RXI: track 0.00 -> 25.1 mm
- net TXO: track 0.00 -> 24.0 mm, vias 0 -> 2
- net GND: track 0.00 -> 23.7 mm, vias 0 -> 5
- net V_BATT: track 0.00 -> 17.7 mm, vias 0 -> 1
- net N_PG: track 0.00 -> 17.3 mm, vias 0 -> 1
- net N$8: track 0.00 -> 17.0 mm, vias 0 -> 1
- net TXLED: track 0.00 -> 13.9 mm
- net RXLED: track 0.00 -> 13.2 mm
- net +3V3: track 0.03 -> 9.91 mm, vias 0 -> 1
- net USBDP: track 0.00 -> 9.85 mm, vias 0 -> 1
- net USBDM: track 0.00 -> 8.88 mm, vias 0 -> 1
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- added copper zone on layer 16, net +3V3
- removed copper zone on layer 16, net 3V3
Other:
- board text added: "10k/THERM"
- board text added: "CHRG"
- board text added: "DONE"
- board text added: "PWR"

Commit message: Yey
Parts:
- moved D1 1.00 mm to (21.0, 7.90)
- moved D2 1.00 mm to (18.7, 7.90)
- moved R1 1.00 mm to (21.0, 7.90)
- moved R2 1.00 mm to (18.7, 7.90)
Routing:
- net GND: track 23.7 -> 18.1 mm
- net N$12: track 0.00 -> 3.26 mm, vias 0 -> 1
- net N$11: track 0.00 -> 3.26 mm, vias 0 -> 1
- net N$10: track 0.00 -> 2.90 mm, vias 0 -> 1
- net N$9: track 0.00 -> 2.88 mm, vias 0 -> 1
- net N$14: track 0.00 -> 2.88 mm, vias 0 -> 1
- net +3V3: track 9.91 -> 11.7 mm
- net USBDM: track 8.88 -> 10.0 mm
- net USBDP: track 9.85 -> 8.97 mm
Other:
- board size 72 x 44 mm -> 65.1 x 35.5 mm
